Commit message: Updated and added new dual_ur5e_allegro_inertia .urdf file variations

File: bimanual-sapien/assets/urdf/ur5e_allegro/robots/dual_ur5e_allegro_inertia_changed_no_collision.urdf (robot description, URDF)
Before this commit: robot dual_ur5e_ability, 57 links, 56 joints
Links:
- link base_link: geometry visual mesh filename=../meshes/dual_ur_stand/base.obj scale=0.044 0.05 0.05
- link forearm_link: geometry visual mesh filename=../meshes/ur5e/visual/forearm.dae
- link forearm_link_r: geometry visual mesh filename=../meshes/ur5e/visual/forearm.dae
- link link_0.0: geometry visual mesh filename=meshes/link_0.0.STL
- link link_0.0_r: geometry visual mesh filename=meshes/link_0.0.STL
- link link_1.0: geometry visual mesh filename=meshes/link_1.0.STL
- link link_1.0_r: geometry visual mesh filename=meshes/link_1.0.STL
- link link_10.0: geometry visual mesh filename=meshes/link_2.0.STL
- link link_10.0_r: geometry visual mesh filename=meshes/link_2.0.STL
- link link_11.0: geometry visual mesh filename=meshes/link_3.0.STL
- link link_11.0_r: geometry visual mesh filename=meshes/link_3.0.STL
- link link_11.0_tip: geometry visual mesh filename=meshes/link_3.0_tip.STL
- link link_11.0_tip_r: geometry visual mesh filename=meshes/link_3.0_tip.STL
- link link_12.0: geometry visual mesh filename=meshes/link_12.0_left.STL
- link link_12.0_r: geometry visual mesh filename=meshes/link_12.0_right.STL
- link link_13.0: geometry visual mesh filename=meshes/link_13.0.STL
- link link_13.0_r: geometry visual mesh filename=meshes/link_13.0.STL
- link link_14.0: geometry visual mesh filename=meshes/link_14.0.STL
- link link_14.0_r: geometry visual mesh filename=meshes/link_14.0.STL
- link link_15.0: geometry visual mesh filename=meshes/link_15.0.STL
- link link_15.0_r: geometry visual mesh filename=meshes/link_15.0.STL
- link link_15.0_tip: geometry visual mesh filename=meshes/link_15.0_tip.STL
- link link_15.0_tip_r: geometry visual mesh filename=meshes/link_15.0_tip.STL
- link link_2.0: geometry visual mesh filename=meshes/link_2.0.STL
- link link_2.0_r: geometry visual mesh filename=meshes/link_2.0.STL
- link link_3.0: geometry visual mesh filename=meshes/link_3.0.STL
- link link_3.0_r: geometry visual mesh filename=meshes/link_3.0.STL
- link link_3.0_tip: geometry visual mesh filename=meshes/link_3.0_tip.STL
- link link_3.0_tip_r: geometry visual mesh filename=meshes/link_3.0_tip.STL
- link link_4.0: geometry visual mesh filename=meshes/link_0.0.STL
- link link_4.0_r: geometry visual mesh filename=meshes/link_0.0.STL
- link link_5.0: geometry visual mesh filename=meshes/link_1.0.STL
- link link_5.0_r: geometry visual mesh filename=meshes/link_1.0.STL
- link link_6.0: geometry visual mesh filename=meshes/link_2.0.STL
- link link_6.0_r: geometry visual mesh filename=meshes/link_2.0.STL
- link link_7.0: geometry visual mesh filename=meshes/link_3.0.STL
- link link_7.0_r: geometry visual mesh filename=meshes/link_3.0.STL
- link link_7.0_tip: geometry visual mesh filename=meshes/link_3.0_tip.STL
- link link_7.0_tip_r: geometry visual mesh filename=meshes/link_3.0_tip.STL
- link link_8.0: geometry visual mesh filename=meshes/link_0.0.STL
- link link_8.0_r: geometry visual mesh filename=meshes/link_0.0.STL
- link link_9.0: geometry visual mesh filename=meshes/link_1.0.STL
- link link_9.0_r: geometry visual mesh filename=meshes/link_1.0.STL
- link shoulder_link: geometry visual mesh filename=../meshes/ur5e/visual/shoulder.dae
- link shoulder_link_r: geometry visual mesh filename=../meshes/ur5e/visual/shoulder.dae
- link upper_arm_link: geometry visual mesh filename=../meshes/ur5e/visual/upperarm.dae
- link upper_arm_link_r: geometry visual mesh filename=../meshes/ur5e/visual/upperarm.dae
- link wrist_1_link: geometry visual mesh filename=../meshes/ur5e/visual/wrist1.dae
- link wrist_1_link_r: geometry visual mesh filename=../meshes/ur5e/visual/wrist1.dae
- link wrist_2_link: geometry visual mesh filename=../meshes/ur5e/visual/wrist2.dae
- link wrist_2_link_r: geometry visual mesh filename=../meshes/ur5e/visual/wrist2.dae
- link wrist_3_link: geometry visual mesh filename=../meshes/ur5e/visual/wrist3.dae
- link wrist_3_link_r: geometry visual mesh filename=../meshes/ur5e/visual/wrist3.dae
- link wrist_base: geometry visual mesh filename=meshes/base_link_left.STL; visual mesh filename=meshes/mount-left.stl scale=0.001 0.001 0.001
- link wrist_base_r: geometry visual mesh filename=meshes/base_link.STL; visual mesh filename=meshes/mount-right.stl scale=0.001 0.001 0.001

File: bimanual-sapien/assets/urdf/ur5e_allegro/robots/dual_ur5e_allegro_inertia_changed_no_hand_collision.urdf (robot description, URDF)
Before this commit: robot dual_ur5e_ability, 57 links, 56 joints
Links:
- link link_0.0: geometry visual mesh filename=meshes/link_0.0.STL
- link link_0.0_r: geometry visual mesh filename=meshes/link_0.0.STL
- link link_1.0: geometry visual mesh filename=meshes/link_1.0.STL
- link link_1.0_r: geometry visual mesh filename=meshes/link_1.0.STL
- link link_10.0: geometry visual mesh filename=meshes/link_2.0.STL
- link link_10.0_r: geometry visual mesh filename=meshes/link_2.0.STL
- link link_11.0: geometry visual mesh filename=meshes/link_3.0.STL
- link link_11.0_r: geometry visual mesh filename=meshes/link_3.0.STL
- link link_11.0_tip: geometry visual mesh filename=meshes/link_3.0_tip.STL
- link link_11.0_tip_r: geometry visual mesh filename=meshes/link_3.0_tip.STL
- link link_12.0: geometry visual mesh filename=meshes/link_12.0_left.STL
- link link_12.0_r: geometry visual mesh filename=meshes/link_12.0_right.STL
- link link_13.0: geometry visual mesh filename=meshes/link_13.0.STL
- link link_13.0_r: geometry visual mesh filename=meshes/link_13.0.STL
- link link_14.0: geometry visual mesh filename=meshes/link_14.0.STL
- link link_14.0_r: geometry visual mesh filename=meshes/link_14.0.STL
- link link_15.0: geometry visual mesh filename=meshes/link_15.0.STL
- link link_15.0_r: geometry visual mesh filename=meshes/link_15.0.STL
- link link_15.0_tip: geometry visual mesh filename=meshes/link_15.0_tip.STL
- link link_15.0_tip_r: geometry visual mesh filename=meshes/link_15.0_tip.STL
- link link_2.0: geometry visual mesh filename=meshes/link_2.0.STL
- link link_2.0_r: geometry visual mesh filename=meshes/link_2.0.STL
- link link_3.0: geometry visual mesh filename=meshes/link_3.0.STL
- link link_3.0_r: geometry visual mesh filename=meshes/link_3.0.STL
- link link_3.0_tip: geometry visual mesh filename=meshes/link_3.0_tip.STL
- link link_3.0_tip_r: geometry visual mesh filename=meshes/link_3.0_tip.STL
- link link_4.0: geometry visual mesh filename=meshes/link_0.0.STL
- link link_4.0_r: geometry visual mesh filename=meshes/link_0.0.STL
- link link_5.0: geometry visual mesh filename=meshes/link_1.0.STL
- link link_5.0_r: geometry visual mesh filename=meshes/link_1.0.STL
- link link_6.0: geometry visual mesh filename=meshes/link_2.0.STL
- link link_6.0_r: geometry visual mesh filename=meshes/link_2.0.STL
- link link_7.0: geometry visual mesh filename=meshes/link_3.0.STL
- link link_7.0_r: geometry visual mesh filename=meshes/link_3.0.STL
- link link_7.0_tip: geometry visual mesh filename=meshes/link_3.0_tip.STL
- link link_7.0_tip_r: geometry visual mesh filename=meshes/link_3.0_tip.STL
- link link_8.0: geometry visual mesh filename=meshes/link_0.0.STL
- link link_8.0_r: geometry visual mesh filename=meshes/link_0.0.STL
- link link_9.0: geometry visual mesh filename=meshes/link_1.0.STL
- link link_9.0_r: geometry visual mesh filename=meshes/link_1.0.STL
- link wrist_1_link: geometry visual mesh filename=../meshes/ur5e/visual/wrist1.dae
- link wrist_1_link_r: geometry visual mesh filename=../meshes/ur5e/visual/wrist1.dae
- link wrist_2_link: geometry visual mesh filename=../meshes/ur5e/visual/wrist2.dae
- link wrist_2_link_r: geometry visual mesh filename=../meshes/ur5e/visual/wrist2.dae
- link wrist_3_link: geometry visual mesh filename=../meshes/ur5e/visual/wrist3.dae
- link wrist_3_link_r: geometry visual mesh filename=../meshes/ur5e/visual/wrist3.dae
- link wrist_base: geometry visual mesh filename=meshes/base_link_left.STL; visual mesh filename=meshes/mount-left.stl scale=0.001 0.001 0.001
- link wrist_base_r: geometry visual mesh filename=meshes/base_link.STL; visual mesh filename=meshes/mount-right.stl scale=0.001 0.001 0.001

File: bimanual-sapien/assets/urdf/ur5e_allegro/robots/dual_ur5e_allegro_inertia_changed_only_hand_collision.urdf (robot description, URDF)
Before this commit: robot dual_ur5e_ability, 57 links, 56 joints
Links:
- link base_link: geometry visual mesh filename=../meshes/dual_ur_stand/base.obj scale=0.044 0.05 0.05
- link forearm_link: geometry visual mesh filename=../meshes/ur5e/visual/forearm.dae
- link forearm_link_r: geometry visual mesh filename=../meshes/ur5e/visual/forearm.dae
- link shoulder_link: geometry visual mesh filename=../meshes/ur5e/visual/shoulder.dae
- link shoulder_link_r: geometry visual mesh filename=../meshes/ur5e/visual/shoulder.dae
- link upper_arm_link: geometry visual mesh filename=../meshes/ur5e/visual/upperarm.dae
- link upper_arm_link_r: geometry visual mesh filename=../meshes/ur5e/visual/upperarm.dae
