Commit message: Added new ur5e_allegro urdf file for only hand collisions not including palm/wrist-base, edited only_hand_collision urdf file to be more accurate

File: bimanual-sapien/assets/urdf/ur5e_allegro/robots/dual_ur5e_allegro_inertia_changed_hand_no_palm_collisions.urdf (robot description, URDF)
Before this commit: robot dual_ur5e_ability, 57 links, 56 joints
Links:
- link wrist_base: geometry visual mesh filename=meshes/base_link_left.STL; visual mesh filename=meshes/mount-left.stl scale=0.001 0.001 0.001
- link wrist_base_r: geometry visual mesh filename=meshes/base_link.STL; visual mesh filename=meshes/mount-right.stl scale=0.001 0.001 0.001
